File: hardware/kicad/gear-miles.kicad_sch (KiCad schematic)
At the start: 53 parts, among them J1 TYPE-C 16PIN 2MD(073), J2 XY-XH2.54-2PWT, J3 UART0 1x4 header, J4 24-pin 0.5 mm FPC, Q1 Si1308EDL, SW1 KH-6X6X5H-STM, SW2 KH-6X6X5H-STM, SW3 KH-6X6X5H-STM, U1 USBLC6-2SC6, U2 ME6217C33P5G, U3 ESP32-C3-WROOM-02-N4

Commit message: fix(hardware): split VSL from PREVGL per GDEY029T94 section 5 p8
- J4.22 (VSL) now on its own net with 1uF/25V bypass C14 and PWR5 flag;
  J4.23 (VGL) keeps PREVGL. Corroborated by native 1:1 raster extraction
  and white-region connectivity trace (different enclosed regions for the
  pin-22 and pin-23 lead stubs).
- Figure diode glyphs render pixel-identically while serving different
  roles, so D2/D3 lead direction remains UNTRACED; pump topology blockers
  stand unchanged and remain marked on-sheet.
- check_blockers PANEL_RAIL_SHORT retained as regression guard; gate now
  exits 3 on five groups (was six).
- Evidence: ERC 0 violations (KiCad 9.0.9), netlist/bounds/blocker-gate/
  pdf-bounds tests pass, raw raster dumps under reports/2026-09-20/.
Parts:
- added C14: 1uF 25V X7R, Gear:TBD_LAYOUT_BLOCKED, symbol Gear:C14_41
- added PWR5: PWR_FLAG, symbol Gear:PWR5_46
- PWR1: symbol Gear:PWR1_41 -> Gear:PWR1_42
- PWR2: symbol Gear:PWR2_42 -> Gear:PWR2_43
- PWR3: symbol Gear:PWR3_43 -> Gear:PWR3_44
- PWR4: symbol Gear:PWR4_44 -> Gear:PWR4_45
- TP1: symbol Gear:TP1_45 -> Gear:TP1_47
- TP2: symbol Gear:TP2_46 -> Gear:TP2_48
- TP3: symbol Gear:TP3_47 -> Gear:TP3_49
- TP4: symbol Gear:TP4_48 -> Gear:TP4_50
- TP5: symbol Gear:TP5_49 -> Gear:TP5_51
- TP6: symbol Gear:TP6_50 -> Gear:TP6_52
- TP7: symbol Gear:TP7_51 -> Gear:TP7_53
- TP8: symbol Gear:TP8_52 -> Gear:TP8_54
- TP9: symbol Gear:TP9_53 -> Gear:TP9_55
Connections:
- net GND: now also C14.2
- net PREVGL: no longer J4.22 (VSL)
- new net VSL: C14.1, J4.22 (VSL), PWR5.1 (PWR)
Other:
- note added: "KNOWN BLOCKER: D2 A=GND/K=PUMP and D3 A=PUMP/K=PREVGL cannot form the intended negative pump (figure leads untraced at native raster resolution). VSL/VGL split applied 2026-09-20 per DS section 5 p8; pump diode and capacitor endpoint audit still required. ERC and netlist tests do not validate analog operation."
- note added: "VSH2 is bypassed to GND through C8 (manufacturer figure C2), never hard-grounded. PWR_FLAGs are limited to USB external rails and panel-derived PREVGH/PREVGL/VSL rails."
- note removed: "KNOWN BLOCKER: D2 A=GND/K=PUMP and D3 A=PUMP/K=PREVGL cannot form the intended negative pump. ERC and netlist tests do not validate analog operation."
- note removed: "VSH2 is bypassed to GND through C8 (manufacturer figure C2), never hard-grounded. PWR_FLAGs are limited to USB external rails and panel-derived PREVGH/PREVGL rails."
- moved on the sheet: PWR1, PWR2, PWR3, PWR4, TP1, TP2, TP3, TP4, TP5, TP6, TP7, TP8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

Commit message: fix(hardware): correct D2/D3 negative-pump polarity per DESPI-C02 vector evidence
Vector-level probe of the official Good Display DESPI-C02_SCH V1.0.pdf
(SHA b1893766...26128b1) resolves the diode-direction question that four
raster passes could not: D1 cathode bar points left (x=645.3..647.7) while
D2/D3 cathode bars point right (x=671.1..673.4), corroborating standard
negative charge-pump topology.

- generate_schematic.py: D2 -> A=PUMP/K=GND clamp, D3 -> A=PREVGL/K=PUMP
  rectifier; on-sheet blocker texts updated to post-correction state
- regenerated gear-miles.kicad_sch (regeneration byte-identical)
- test_netlist.py: CRITICAL_EXPECTED updated with the source change
- check_blockers.py: polarity checks retained as regression guards, basis
  text now cites the vector probe; gate now exits 3 on three groups (was
  five) - NEGATIVE_PUMP_* cleared
- docs/schematic.md: blocking-findings row, netlist-test note, and new
  2026-09-28 addendum; report summary updated
- reports/2026-09-28: ERC (0 violations) and blocker JSON refreshed

Static reference-design corroboration only - no simulation, no bench.
Design remains not-for-build; 17 identity, 21 footprint, 41 verification
blockers and the panel endpoint map remain open.
Connections:
- net GND: now also D2.1 (K); no longer D2.2 (A)
- net PREVGL: now also D3.2 (A); no longer D3.1 (K)
- net PUMP: now also D2.2 (A), D3.1 (K); no longer D2.1 (K), D3.2 (A)
Other:
- note added: "KNOWN BLOCKER (CORRECTED 2026-09-28): D2 (A=PUMP, K=GND clamp) and D3 (A=PREVGL, K=PUMP rectifier) orientations corrected to standard negative charge pump topology, corroborated by Good Display DESPI-C02 V1.0 vector schematic. VSL/VGL split applied 2026-09-20 per DS section 5 p8; ERC and netlist tests pass."
- note added: "NOT FOR FABRICATION OR POWER-UP: REJECTED CANDIDATE. Pump diode polarity corrected 2026-09-28; panel capacitor endpoints, unresolved identities and placeholder footprints remain blocked pending independent review."
- note removed: "KNOWN BLOCKER: D2 A=GND/K=PUMP and D3 A=PUMP/K=PREVGL cannot form the intended negative pump (figure leads untraced at native raster resolution). VSL/VGL split applied 2026-09-20 per DS section 5 p8; pump diode and capacitor endpoint audit still required. ERC and netlist tests do not validate analog operation."
- note removed: "NOT FOR FABRICATION OR POWER-UP: REJECTED CANDIDATE. Pump diode polarity and panel capacitor endpoints require correction and independent manufacturer-diagram review."
Changed lines of the file:
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@@
     (rev "Issue 3 - BLOCKED")
     (company "Gear Miles"))
-  (text "NOT FOR FABRICATION OR POWER-UP: REJECTED CANDIDATE. Pump diode polarity and panel capacitor endpoints require correction and independent manufacturer-diagram review." (exclude_from_sim no) (at 45 555 0)
+  (text "NOT FOR FABRICATION OR POWER-UP: REJECTED CANDIDATE. Pump diode polarity corrected 2026-09-28; panel capacitor endpoints, unresolved identities and placeholder footprints remain blocked pending independent review." (exclude_from_sim no) (at 45 555 0)
     (effects (font (size 1.27 1.27)) (justify left bottom)))
-  (text "KNOWN BLOCKER: D2 A=GND/K=PUMP and D3 A=PUMP/K=PREVGL cannot form the intended negative pump (figure leads untraced at native raster resolution). VSL/VGL split applied 2026-09-20 per DS section 5 p8; pump diode and capacitor endpoint audit still required. ERC and netlist tests do not validate analog operation." (exclude_from_sim no) (at 45 563 0)
+  (text "KNOWN BLOCKER (CORRECTED 2026-09-28): D2 (A=PUMP, K=GND clamp) and D3 (A=PREVGL, K=PUMP rectifier) orientations corrected to standard negative charge pump topology, corroborated by Good Display DESPI-C02 V1.0 vector schematic. VSL/VGL split applied 2026-09-20 per DS section 5 p8; ERC and netlist tests pass." (exclude_from_sim no) (at 45 563 0)
     (effects (font (size 1.27 1.27)) (justify left bottom)))
   (text "VSH2 is bypassed to GND through C8 (manufacturer figure C2), never hard-grounded. PWR_FLAGs are limited to USB external rails and panel-derived PREVGH/PREVGL/VSL rails." (exclude_from_sim no) (at 45.72 571.5 0)
@@
     (pin "2")
   )
-  (global_label "PUMP" (shape input) (at 129.54 322.58 0) (effects (font (size 1.0 1.0))))
-  (global_label "GND" (shape input) (at 129.54 325.12 0) (effects (font (size 1.0 1.0))))
+  (global_label "GND" (shape input) (at 129.54 322.58 0) (effects (font (size 1.0 1.0))))
+  (global_label "PUMP" (shape input) (at 129.54 325.12 0) (effects (font (size 1.0 1.0))))
   (symbol (lib_id "Gear:D3_30") (at 238.76 325.12 0) (unit 1)
     (exclude_from_sim no) (in_bom yes) (on_board yes)
@@
     (pin "2")
   )
-  (global_label "PREVGL" (shape input) (at 231.14 322.58 0) (effects (font (size 1.0 1.0))))
-  (global_label "PUMP" (shape input) (at 231.14 325.12 0) (effects (font (size 1.0 1.0))))
+  (global_label "PUMP" (shape input) (at 231.14 322.58 0) (effects (font (size 1.0 1.0))))
+  (global_label "PREVGL" (shape input) (at 231.14 325.12 0) (effects (font (size 1.0 1.0))))
   (symbol (lib_id "Gear:D4_31") (at 340.35999999999996 325.12 0) (unit 1)
     (exclude_from_sim no) (in_bom yes) (on_board yes)
